File: kicad_board/termint-wifi.kicad_pcb (KiCad board)
At the start: 2 copper layers, 118.9 x 33.9 mm, 20 parts, among them J1 Conn_01x04_Male, J2 Conn_01x08, J3 Conn_01x08

Commit message: Updated component numbering
Parts:
- renumbered C7 to C3, WEMOS to WEMOS_D1
Other:
- board text added: "WEMOS"
